Commit message: Classic wheels mode with efforts feedback (alfa)

File: urdf/youbot_base/base.gazebo.xacro (robot description, xacro)
@@ -14,7 +14,4 @@
       <kd>100</kd>
     </gazebo>
-    <gazebo reference="caster_link_fl">
-      <material value="youbot/Orange" />
-    </gazebo>
     <!-- front right wheel -->
     <gazebo reference="wheel_link_fr">
@@ -22,7 +19,4 @@
       <kp>1000000</kp>
       <kd>100</kd>
-    </gazebo>
-    <gazebo reference="caster_link_fr">
-      <material value="youbot/Orange" />
     </gazebo>
     <!-- back left wheel -->
@@ -32,7 +26,4 @@
       <kd>100</kd>
     </gazebo>
-    <gazebo reference="caster_link_bl">
-      <material value="youbot/Orange" />
-    </gazebo>
     <!-- back right wheel -->
     <gazebo reference="wheel_link_br">
@@ -41,10 +32,7 @@
       <kd>100</kd>
     </gazebo>
-    <gazebo reference="caster_link_br">
-      <material value="youbot/Orange" />
-    </gazebo>
     <!-- position controller -->
     <gazebo>
-      <plugin name="base_controller" filename="libgazebo_ros_planar_move.so">
+      <!--plugin name="base_controller" filename="libgazebo_ros_planar_move.so">
         <commandTopic>cmd_vel</commandTopic>
         <odometryTopic>odom</odometryTopic>
@@ -52,5 +40,5 @@
         <odometryRate>100.0</odometryRate>
         <robotBaseFrame>base_footprint</robotBaseFrame>
-      </plugin>
+      </plugin-->
     </gazebo>
   </xacro:macro>

File: urdf/youbot_base/base.transmission.xacro (robot description, xacro)
@@ -4,6 +4,5 @@
        xmlns:interface="http://playerstage.sourceforge.net/gazebo/xmlschema/#interface"
        xmlns:xacro="http://ros.org/wiki/xacro">
-	<xacro:property name="wheel_mechanical_reduction" value="${624/35 * 80/18}" />
-	<xacro:property name="caster_mechanical_reduction" value="${624/35 * 80/18}" />
+	<xacro:property name="wheel_mechanical_reduction" value="1" />
 	<xacro:macro name="youbot_base_transmission">
 	<!-- front left wheel -->
@@ -11,84 +10,44 @@
       <type>transmission_interface/SimpleTransmission</type>
 			<actuator name="wheel_motor_fl">
-        <hardwareInterface>VelocityJointInterface</hardwareInterface>
+        <hardwareInterface>hardware_interface/EffortJointInterface</hardwareInterface>
         <mechanicalReduction>${wheel_mechanical_reduction}</mechanicalReduction>
       </actuator>
 			<joint name="wheel_joint_fl">
-        <hardwareInterface>VelocityJointInterface</hardwareInterface>
+        <hardwareInterface>hardware_interface/EffortJointInterface</hardwareInterface>
       </joint>
 		</transmission>
-		<transmission name="caster_trans_fl">
-      <type>transmission_interface/SimpleTransmission</type>
-   	  <actuator name="caster_motor_fl">
-        <hardwareInterface>VelocityJointInterface</hardwareInterface>
-        <mechanicalReduction>${caster_mechanical_reduction}</mechanicalReduction>
-      </actuator>
-      <joint name="caster_joint_fl">
-        <hardwareInterface>VelocityJointInterface</hardwareInterface>
-      </joint>
-    </transmission>
 	  <!-- front right wheel -->
 	  <transmission name="wheel_trans_fr">
       <type>transmission_interface/SimpleTransmission</type>
 		  <actuator name="wheel_motor_fr">
-        <hardwareInterface>VelocityJointInterface</hardwareInterface>
+        <hardwareInterface>hardware_interface/EffortJointInterface</hardwareInterface>
         <mechanicalReduction>${wheel_mechanical_reduction}</mechanicalReduction>
       </actuator>
 		  <joint name="wheel_joint_fr">
-        <hardwareInterface>VelocityJointInterface</hardwareInterface>
+        <hardwareInterface>hardware_interface/EffortJointInterface</hardwareInterface>
       </joint>
 	  </transmission>
-	  <transmission name="caster_trans_fr">
-      <type>transmission_interface/SimpleTransmission</type>
-      <actuator name="caster_motor_fr" >
-        <hardwareInterface>VelocityJointInterface</hardwareInterface>
-        <mechanicalReduction>${caster_mechanical_reduction}</mechanicalReduction>
-      </actuator>
-      <joint name="caster_joint_fr">
-        <hardwareInterface>VelocityJointInterface</hardwareInterface>
-      </joint>
-    </transmission>
 	  <!-- back left wheel -->
 	  <transmission name="wheel_trans_bl">
       <type>transmission_interface/SimpleTransmission</type>
 	    <actuator name="wheel_motor_bl" >
-        <hardwareInterface>VelocityJointInterface</hardwareInterface>
+        <hardwareInterface>hardware_interface/EffortJointInterface</hardwareInterface>
         <mechanicalReduction>${wheel_mechanical_reduction}</mechanicalReduction>
       </actuator>
 	    <joint name="wheel_joint_bl">
-        <hardwareInterface>VelocityJointInterface</hardwareInterface>
+        <hardwareInterface>hardware_interface/EffortJointInterface</hardwareInterface>
       </joint>
 	  </transmission>
-	  <transmission name="caster_trans_bl">
-      <type>transmission_interface/SimpleTransmission</type>
-      <actuator name="caster_motor_bl" >
-        <hardwareInterface>VelocityJointInterface</hardwareInterface>
-        <mechanicalReduction>${caster_mechanical_reduction}</mechanicalReduction>
-      </actuator>
-      <joint name="caster_joint_bl">
-        <hardwareInterface>VelocityJointInterface</hardwareInterface>
-      </joint>
-    </transmission>
 	  <!-- back right wheel -->
 	  <transmission name="wheel_trans_br">
       <type>transmission_interface/SimpleTransmission</type>
 	    <actuator name="wheel_motor_br" >
-        <hardwareInterface>VelocityJointInterface</hardwareInterface>
+        <hardwareInterface>hardware_interface/EffortJointInterface</hardwareInterface>
         <mechanicalReduction>${wheel_mechanical_reduction}</mechanicalReduction>
       </actuator>
 		  <joint name="wheel_joint_br">
-        <hardwareInterface>VelocityJointInterface</hardwareInterface>
+        <hardwareInterface>hardware_interface/EffortJointInterface</hardwareInterface>
       </joint>
 	  </transmission>
-	  <transmission name="caster_trans_br">
-      <type>transmission_interface/SimpleTransmission</type>
-      <actuator name="caster_motor_br" >
-        <hardwareInterface>VelocityJointInterface</hardwareInterface>
-        <mechanicalReduction>${caster_mechanical_reduction}</mechanicalReduction>
-      </actuator>
-      <joint name="caster_joint_br">
-        <hardwareInterface>VelocityJointInterface</hardwareInterface>
-      </joint>
-    </transmission>
   </xacro:macro>
 </robot>

File: urdf/youbot_base/base.urdf.xacro (robot description, xacro)
@@ -80,5 +80,5 @@
     </link>
     <!-- front left wheel -->
-    <joint name="caster_joint_fl" type="continuous">
+    <joint name="caster_joint_fl" type="fixed">
       <origin xyz="${caster_offset_x} ${caster_offset_y} ${caster_offset_z}" rpy="0 0 0"/>
       <axis xyz="0 0 1"/>
@@ -127,5 +127,5 @@
     </link>
     <!-- front right wheel -->
-    <joint name="caster_joint_fr" type="continuous">
+    <joint name="caster_joint_fr" type="fixed">
       <origin xyz="${caster_offset_x} ${-caster_offset_y} ${caster_offset_z}" rpy="0 0 0"/>
       <axis xyz="0 0 1"/>
@@ -174,5 +174,5 @@
     </link>
     <!-- back left wheel -->
-    <joint name="caster_joint_bl" type="continuous">
+    <joint name="caster_joint_bl" type="fixed">
       <origin xyz="${-caster_offset_x} ${caster_offset_y} ${caster_offset_z}" rpy="0 0 0"/>
       <axis xyz="0 0 1"/>
@@ -222,5 +222,5 @@
     </link>
     <!-- back right wheel -->
-    <joint name="caster_joint_br" type="continuous">
+    <joint name="caster_joint_br" type="fixed">
       <origin xyz="${-caster_offset_x} ${-caster_offset_y} ${caster_offset_z}" rpy="0 0 0"/>
       <axis xyz="0 0 1"/>
